File: AVRISP2TC/AVRISP2TC.brd (EAGLE design)
At the start: 39.4 x 34 mm, 13 parts, among them U1 NCP1117LPST33T3G

Commit message: Added AVRISP2TC
Parts:
- removed SI_PROGRAMMER: 5103308-1, PP_Connectors:5103308-1
- added 10PIN_ISP: 5103308-1, PP_Connectors:5103308-1
- added 6PIN_ISP: 30306-6002HB, PP_Connectors:30306-6002HB
- moved FRAME1 20.7 mm to (10.2, 25.1), turned to 0 degrees
- moved TC2030 0.40 mm to (33.7, 10.8)
- renumbered C2 to C3
Connections:
- removed net !RST!/C2CK: SI_PROGRAMMER.7, TC2030.3
- removed net C2D: SI_PROGRAMMER.4, TC2030.4
- new net MISO: 10PIN_ISP.1, 6PIN_ISP.1, TC2030.1
- new net MOSI: 10PIN_ISP.9, 6PIN_ISP.4, TC2030.4
- new net RST: 10PIN_ISP.5, 6PIN_ISP.5, TC2030.5
- new net SCK: 10PIN_ISP.7, 6PIN_ISP.3, TC2030.3
- net GND: now also 10PIN_ISP.10, 10PIN_ISP.4, 10PIN_ISP.6, 10PIN_ISP.8, 6PIN_ISP.6, TC2030.6; no longer SI_PROGRAMMER.2, SI_PROGRAMMER.3, TC2030.1
- net VCC: now also 10PIN_ISP.2, 6PIN_ISP.2
Routing:
- net MOSI: track 0.00 -> 46.8 mm
- net VCC: track 35.9 -> 81.7 mm
- net SCK: track 0.00 -> 42.5 mm
- net RST: track 0.00 -> 35.6 mm
- net MISO: track 0.00 -> 33.2 mm
- net !RST!/C2CK: track 32.0 -> 0.00 mm
- net C2D: track 27.0 -> 0.00 mm

Commit message: Pushing Camfiles
Parts:
- turned U1 to 180 degrees
Changed lines of the file:
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@@
 <attribute name="VALUE" value="MF-CON-MICROUSB-RIGHT" x="2.921" y="28.575" size="1.778" layer="27" rot="R270" display="off"/>
 </element>
-<element name="U1" library="MF_IC_Power" package="SOT-223-3" value="NCP1117LPST33T3G" x="28.575" y="28.575" smashed="yes" rot="R90">
-<attribute name="NAME" x="23.821" y="26.341" size="1.27" layer="25" font="vector" ratio="16" rot="R90"/>
-<attribute name="MPN" value="NCP1117LPST33T3G" x="28.575" y="28.575" size="1.778" layer="27" rot="R90" display="off"/>
-<attribute name="HOUSEPART" value="NO" x="28.575" y="28.575" size="1.778" layer="27" rot="R90" display="off"/>
-<attribute name="POPULATE" value="1" x="28.575" y="28.575" size="1.778" layer="27" rot="R90" display="off"/>
-<attribute name="URL" value="http://www.onsemi.com/pub_link/Collateral/NCP1117LP-D.PDF" x="28.575" y="28.575" size="1.778" layer="27" rot="R90" display="off"/>
-<attribute name="VALUE" value="NCP1117LPST33T3G" x="28.575" y="28.575" size="1.778" layer="27" rot="R90" display="off"/>
+<element name="U1" library="MF_IC_Power" package="SOT-223-3" value="NCP1117LPST33T3G" x="28.575" y="28.575" smashed="yes" rot="R180">
+<attribute name="NAME" x="30.809" y="23.821" size="1.27" layer="25" font="vector" ratio="16" rot="R180"/>
+<attribute name="MPN" value="NCP1117LPST33T3G" x="28.575" y="28.575" size="1.778" layer="27" rot="R180" display="off"/>
+<attribute name="HOUSEPART" value="NO" x="28.575" y="28.575" size="1.778" layer="27" rot="R180" display="off"/>
+<attribute name="POPULATE" value="1" x="28.575" y="28.575" size="1.778" layer="27" rot="R180" display="off"/>
+<attribute name="URL" value="http://www.onsemi.com/pub_link/Collateral/NCP1117LP-D.PDF" x="28.575" y="28.575" size="1.778" layer="27" rot="R180" display="off"/>
+<attribute name="VALUE" value="NCP1117LPST33T3G" x="28.575" y="28.575" size="1.778" layer="27" rot="R180" display="off"/>
 </element>
 <element name="F1" library="PP_Passives" package="1206" value="0ZCJ0010FF2E" x="9.525" y="30.353" rot="R90">
@@
 <attribute name="VALUE" value="" x="36.195" y="26.67" size="1.778" layer="27" rot="R180" display="off"/>
 </element>
-<element name="U$3" library="PP_Aesthetics" package="MF_LOGO_MEDIUM" value="MF_LOGOLOGO_MEDIUM" x="28.194" y="7.112" rot="R90"/>
+<element name="U$3" library="PP_Aesthetics" package="MF_LOGO_MEDIUM" value="MF_LOGOLOGO_MEDIUM" x="28.194" y="7.112" rot="R90">
+<attribute name="POPULATE" value="0" x="28.194" y="7.112" size="1.778" layer="27" rot="R90" display="off"/>
+<attribute name="MPN" value="" x="28.194" y="7.112" size="1.778" layer="27" rot="R90" display="off"/>
+</element>
 <element name="C1" library="MF_Passives" package="C1206" value="10uF" x="15.24" y="27.305" smashed="yes" rot="R180">
 <attribute name="TOLERANCE" value="" x="15.24" y="27.305" size="1.778" layer="27" rot="R180" display="off"/>
